File: PC-370_P.sch (KiCad schematic (older format))
At the start: 75 parts, among them J1 MEMORY CONNECTION, U1 74LS373, U10 74LS20, U11 74LS138, U12 74LS138, U13 74LS138, U14 74LS138, U15 74LS175, U16 74LS112, U17 74LS175, U18 74LS112, U19 74LS175, U2 74LS245, U20 74LS112, U21 74LS125, U22 74LS153, U24 INTEL 287, U25 74LS245, U26 74LS245, U27 74LS373, U28 74LS373, U29 74LS373, U3 74LS245, U30 74LS245, U31 MCM2114P, U32 74LS27, U33 74LS10, U34 74LS00, U35 74LS74, U36 74LS09, U37 74LS02, U38 74LS08, U39 74LS74, U4 74LS373, U40 74LS27, U41 74LS08, U42 74LS32, U43 74LS02, U44 74LS157, U45 74LS153, U46 74LS153, U47 314A472, U48 74LS10, U49 74LS10, U5 74LS373, U50 74LS04, U51 74LS08, U52 74LS00, U53 74LS30, U54 74LS74, U55 74LS153, U56 74LS04, U57 74LS30, U58 74LS157, U59 74LS00, U6 74LS374, U60 74LS04, U61 74LS157, U62 68000-PGA, U63 68000-PGA, U64 MCM2114P, U65 MCM2114P, U66 74LS280, U67 74LS32, U68 74LS00, U69 74LS74, U7 74LS244, U70 74LS74, U71 74LS86, U72 74LS32, U73 74LS04, U74 74LS02, U8 74LS241, U9 74LS30

Commit message: Migrated work from spreadsheet, original numbered net names used.
Parts:
- added J?: Bus_ISA_8bit, symbol Connector:Bus_ISA_8bit
- gave numbers to parts that had none: 1
Connections:
- net ##88: now reaches U1.1 (OE)
- net ##88: now also U14.14 (O1)
- net ##89: now reaches U1.2 (O0)
- net ##89: now also J1.19 (Pin_19), U2.2 (A0), U3.2 (A0), U4.2 (O0), U4.3 (D0), U5.2 (O0), U6.2 (O0), U7.2 (I0a), U8.18 (O0a)
- net ##90: now reaches U1.3 (D0)
- net ##90: now also U24.6 (Pin_6), U62.J2 (IPL0)
- net ##91: now reaches U1.4 (D1)
- net ##91: now also U20.7 (~Q), U62.H3 (IPL1)
- net ##92: now reaches U1.5 (O1)
- net ##92: now also J1.20 (Pin_20), U2.3 (A1), U3.3 (A1), U4.18 (D7), U4.19 (O7), U43.11, U5.19 (O7), U6.19 (O7), U7.4 (I1a), U8.16 (O1a)
- net ##93: now reaches U1.8 (D3)
- net ##93: now also U20.5 (Q), U21.5
- net ##94: now reaches U1.9 (O3)
- net ##94: now also J1.26 (Pin_26), U2.9 (A7), U3.9 (A7), U4.12 (O4), U4.13 (D4), U43.2, U5.12 (O4), U6.12 (O4), U8.12 (O3a)
- net ##83: now reaches U2.1 (A->B)
- net ##83: now also U24.7 (Pin_7), U25.1 (A->B), U74.10
- net ##87: now reaches U3.19 (CE)
- net ##87: now also U26.19 (CE), U67.13, U67.4, U68.2, U73.2
- net ##36: now reaches U5.13 (D4)
- net ##36: now also U31.4 (Pin_4), U32.2, U42.13, U62.G9 (A15), U63.G9 (A15), U64.4 (Pin_4), U65.4 (Pin_4)
- net ##34: now reaches U5.14 (D5)
- net ##34: now also U31.6 (Pin_6), U32.1, U44.11 (I0c), U62.H8 (A13), U63.H8 (A13), U64.6 (Pin_6), U65.6 (Pin_6)
- net ##68: now reaches U5.3 (D0)
- net ##68: now also U45.13 (I3b), U62.J7 (A8), U63.J7 (A8), U9.1, U9.5
- net ##33: now reaches U5.7 (D2)
- net ##33: now also U31.5 (Pin_5), U44.14 (I0d), U62.H9 (A12), U63.H9 (A12), U64.5 (Pin_5), U65.5 (Pin_5), U9.6
- net ##35: now reaches U5.8 (D3)
- net ##35: now also U31.7 (Pin_7), U44.5 (I0b), U62.J10 (A14), U63.J10 (A14), U64.7 (Pin_7), U65.7 (Pin_7), U9.11
- net ##31: now reaches U7.15 (I2b)
- net ##31: now also U47.2 (Pin_2), U54.10 (~S), U54.13 (~R), U55.12 (I2b), U55.13 (I3b), U55.3 (I3a), U55.4 (I2a)
- net ##32: now reaches U7.16 (O1a)
- net ##32: now also U64.12 (Pin_12), U7.5 (O2b)
- net ##8: now reaches U8.13 (I1b)
- net ##8: now also U19.10 (Q2)
- net ##10: now reaches U8.3 (O3b)
- net ##10: now also U69.3 (C)
- net #32: now reaches U8.4 (I1a)
- net ##60: now reaches U8.9 (O0b)
- net ##60: now also U20.1 (C), U20.13 (C), U24.13 (Pin_13)
- net ##86: now reaches U11.12 (O3)
- net ##86: now also U40.1, U40.3, U48.4, U73.1
- net ##74: now reaches U12.1 (A0)
- net ##74: now also U13.1 (A0), U14.1 (A0), U22.13 (I3b), U28.7 (D2), U62.K6 (A4), U63.K6 (A4)
- net ##84: now reaches U12.13 (O2)
- net ##84: now also U74.11
- net ##79: now reaches U12.14 (O1)
- net ##79: now also U74.5
- net ##69: now reaches U12.2 (A1)
- net ##69: now also U13.2 (A1), U14.2 (A1), U28.14 (D5), U46.3 (I3a), U62.J6 (A5), U63.J6 (A5)
- net ##70: now reaches U12.3 (A2)
- net ##70: now also U13.3 (A2), U14.3 (A2), U28.8 (D3), U46.13 (I3b), U62.K7 (A6), U63.K7 (A6)
- net ##63: now reaches U13.14 (O1)
- net ##63: now also U43.12, U43.3
- net ##7: now reaches U19.11 (~Q2)
- net ##7: now also U24.15 (Pin_15)
- net ISA_DB0: now reaches U19.12 (D2)
- net ISA_DB0: now also J?.40 (DB0)
- net ISA_DB2: now reaches U19.13 (D3)
- net ISA_DB2: now also J?.38 (DB2)
- net ##6: now reaches U19.14 (~Q3)
- net ##6: now also U21.4
- net ##28: now reaches U19.2 (Q0)
- net ##28: now also U55.14 (S0)
- net ISA_DB3: now reaches U19.4 (D0)
- net ISA_DB3: now also J?.37 (DB3)
- net ISA_DB1: now reaches U19.5 (D1)
- net ISA_DB1: now also J?.39 (DB1)
- net ##14: now reaches U19.9 (Cp)
- net ##14: now also U59.3
- net ##23: now reaches U20.2 (K)
- net ##23: now also U51.11
- net ##61: now reaches U20.3 (J)
- net ##61: now also U43.1
- net ##22: now reaches U20.11 (J)
- net ##22: now also U41.11
- net ##62: now reaches U20.12 (K)
- net ##62: now also U43.13
- net ##25: now reaches U20.9 (Q)
- net ##25: now also U21.2
- net ##24: now reaches U21.1
- net ##24: now also U42.3
- net ISA_DB7: now reaches U21.3
- net ISA_DB7: now also J?.33 (DB7)
- net ISA_BA00_BUFF: now reaches U21.8
- net ISA_BA00_BUFF: now also U59.12, U59.2, U60.5, U61.11 (I0c)
- net ISA_BA00: now reaches U21.9
- net ISA_BA00: now also J?.62 (BA00)
- net ISA_BA12: now reaches U22.10 (I0b)
- net ISA_BA12: now also J?.50 (BA12)
- net ISA_BA04: now reaches U22.11 (I1b)
- net ISA_BA04: now also U57.6, J?.58 (BA04)
- net ##73: now reaches U22.3 (I3a)
- net ##73: now also U28.4 (D1), U62.K5 (A3), U63.K5 (A3)
- net ISA_BA03: now reaches U22.5 (I1a)
- net ISA_BA03: now also U56.9, J?.59 (BA03)
- net ISA_BA11: now reaches U22.6 (I0a)
- net ISA_BA11: now also J?.51 (BA11)
- net ##49: now reaches U22.7 (Za)
- net ##49: now also J1.4 (Pin_4)
- net ##50: now reaches U22.9 (Zb)
- net ##50: now also J1.5 (Pin_5)
- net ISA_BA10: now reaches U23.10 (I0b)
- net ISA_BA10: now also J?.52 (BA10)
- net ISA_BA02: now reaches U23.11 (I1b)
- net ISA_BA02: now also U51.13, J?.60 (BA02)
- net ##72: now reaches U23.13 (I3b)
- net ##72: now also U28.17 (D6), U62.J5 (A2), U63.J5 (A2)
- net ##71: now reaches U23.3 (I3a)
- net ##71: now also U28.18 (D7), U62.K4 (A1), U63.K4 (A1), U74.12
- net ISA_BA01: now reaches U23.5 (I1a)
- net ISA_BA01: now also U41.13, J?.61 (BA01)
- net ISA_BA09: now reaches U23.6 (I0a)
- net ISA_BA09: now also U57.11, J?.53 (BA09)
- net ##47: now reaches U23.7 (Za)
- net ##47: now also J1.2 (Pin_2)
- net ##48: now reaches U23.9 (Zb)
- net ##48: now also J1.3 (Pin_3)
- net ##75: now reaches U24.8 (Pin_8)
- net ##75: now also U74.1
- net ##67: now reaches U28.13 (D4)
- net ##67: now also U45.3 (I3a), U62.K8 (A7), U63.K8 (A7)
- net ##42: now reaches U29.14 (D5)
- net ##42: now also U31.15 (Pin_15), U62.D10 (A21), U63.D10 (A21), U64.15 (Pin_15), U65.15 (Pin_15)
- net ##39: now reaches U29.17 (D6)
- net ##39: now also U31.1 (Pin_1), U42.9, U62.F9 (A18), U63.F9 (A18), U64.1 (Pin_1), U65.1 (Pin_1)
- net ##38: now reaches U29.18 (D7)
- net ##38: now also U31.2 (Pin_2), U62.G10 (A17), U63.G10 (A17), U64.2 (Pin_2), U65.2 (Pin_2), U67.2
- net ##37: now reaches U29.3 (D0)
- net ##37: now also U31.3 (Pin_3), U42.4, U62.H10 (A16), U63.H10 (A16), U64.3 (Pin_3), U65.3 (Pin_3)
- net ##40: now reaches U29.4 (D1)
- net ##40: now also U31.17 (Pin_17), U62.F10 (A19), U63.F10 (A19), U64.17 (Pin_17), U65.17 (Pin_17)
- net ##41: now reaches U29.7 (D2)
- net ##41: now also U31.16 (Pin_16), U62.E10 (A20), U63.E10 (A20), U64.16 (Pin_16), U65.16 (Pin_16)
- net ##57: now reaches U30.2 (A0)
- net ##57: now also U31.14 (Pin_14), U44.13 (I1d), U66.11 (D)
- net ##56: now reaches U30.3 (A1)
- net ##56: now also U31.13 (Pin_13), U44.10 (I1c), U66.10 (C)
- net ##59: now reaches U30.4 (A2)
- net ##59: now also U31.12 (Pin_12), U44.6 (I1b), U66.9 (B)
- net ##58: now reaches U30.5 (A3)
- net ##58: now also U31.11 (Pin_11), U44.3 (I1a), U66.8 (A)
- net ##78: now reaches U32.11
- net ##78: now also U74.4
- net ##46: now reaches U37.9
- net ##46: now also U42.10, U42.12, U42.5, U49.12, U67.1
- net ##76: now reaches U40.6
- net ##76: now also U74.2
- net ##82: now reaches U40.8
- net ##82: now also U74.9
- net ##15: now reaches U41.12
- net ##15: now also U43.4, U51.12, U59.1
- net ##16: now reaches U42.2
- net ##16: now also U43.6, U57.8
- net ##45: now reaches U42.6
- net ##45: now also U58.14 (I0d)
- net ##44: now reaches U42.8
- net ##44: now also U58.5 (I0b)
- net ##43: now reaches U42.11
- net ##43: now also U44.2 (I0a)
- net ##65: now reaches U44.4 (Za)
- net ##65: now also U45.4 (I2a)
- net ##64: now reaches U44.7 (Zb)
- net ##64: now also U46.12 (I2b)
- net ##55: now reaches U44.9 (Zc)
- net ##55: now also U46.4 (I2a)
- net ISA_BA16: now reaches U45.10 (I0b)
- net ISA_BA16: now also J?.46 (BA16)
- net ISA_BA08: now reaches U45.11 (I1b)
- net ISA_BA08: now also U57.12, J?.54 (BA08)
- net ##66: now reaches U45.12 (I2b)
- net ##66: now also U58.12 (Zd)
- net EFFECTIVE_ISA_A07: now reaches U45.5 (I1a)
- net EFFECTIVE_ISA_A07: now also U59.8
- net ISA_BA15: now reaches U45.6 (I0a)
- net ISA_BA15: now also J?.47 (BA15)
- net ##53: now reaches U45.7 (Za)
- net ##53: now also J1.8 (Pin_8)
- net ##54: now reaches U45.9 (Zb)
- net ##54: now also J1.9 (Pin_9)
- net ISA_BA14: now reaches U46.10 (I0b)
- net ISA_BA14: now also J?.48 (BA14)
- net ISA_BA06: now reaches U46.11 (I1b)
- net ISA_BA06: now also U56.11, J?.56 (BA06)
- net ISA_BA05: now reaches U46.5 (I1a)
- net ISA_BA05: now also U57.5, J?.57 (BA05)
- net ISA_BA13: now reaches U46.6 (I0a)
- net ISA_BA13: now also J?.49 (BA13)
- net ##51: now reaches U46.7 (Za)
- net ##51: now also J1.6 (Pin_6)
- net ##52: now reaches U46.9 (Zb)
- net ##52: now also J1.7 (Pin_7)
- net ##80: now reaches U54.9 (Q)
- net ##80: now also U74.6
- net ISA_BA17: now reaches U55.10 (I0b)
- net ISA_BA17: now also U55.5 (I1a), J?.45 (BA17)
- net ISA_BA19: now reaches U55.2 (S1)
- net ISA_BA19: now also J?.43 (BA19)
- net ##26: now reaches U55.7 (Za)
- net ##26: now also U61.5 (I0b)
- net ##27: now reaches U55.9 (Zb)
- net ##27: now also U61.2 (I0a)
- net at U56.8: now also U57.4
- net at U56.10: now also U57.3
- net at U56.12: now also U57.2
- net ISA_BA07: now reaches U56.13
- net ISA_BA07: now also U59.4, J?.55 (BA07)
- net ~ISA_AEN: now reaches U57.1
- net ~ISA_AEN: now also U60.12
- net at U59.10: now also U59.11
- net at U59.9: now also U59.6
- net ~ISA_REFRESH: now reaches U59.5
- net ~ISA_REFRESH: now also U60.1, J?.19 (~DACK0)
- net ISA_REFRESH: now reaches U59.13
- net ISA_REFRESH: now also U60.2
- net ~ISA_BA00: now reaches U60.6
- net ISA_AEN: now reaches U60.13
- net ISA_AEN: now also J?.42 (AEN)
- net ##29: now reaches U61.4 (Za)
- net ##29: now also J1.28 (Pin_28)
- net ##30: now reaches U61.7 (Zb)
- net ##30: now also J1.29 (Pin_29)
- net ##85: now reaches U67.12
- net ##85: now also U74.13
- net ##81: now reaches U73.6
- net ##81: now also U74.8
- net ##77: now reaches U73.12
- net ##77: now also U74.3
Other:
- moved on the sheet: U21A, U21B, U21D

Commit message: Finished tracing out the board
Connections:
- net ##32: now also U71.1
- net ~ISA_BA00: now also U61.14 (I0d)
- net ##108: now reaches U1.11 (LE)
- net ##108: now also U18.1 (C), U32.5, U39.3 (C), U69.2 (D), U69.6 (~Q), U70.11 (C)
- net ##107: now reaches U1.12 (O4)
- net ##107: now also J1.18 (Pin_18), U25.9 (A7), U26.9 (A7), U27.12 (O4), U27.13 (D4), U28.12 (O4), U29.12 (O4)
- net ##99: now reaches U1.13 (D4)
- net ##99: now also U24.5 (Pin_5), U54.12 (D)
- net ##98: now reaches U1.14 (D5)
- net ##98: now also U18.3 (J), U24.4 (Pin_4)
- net ##106: now reaches U1.15 (O5)
- net ##106: now also J1.17 (Pin_17), U25.8 (A6), U26.8 (A6), U27.8 (D3), U27.9 (O3), U28.9 (O3), U29.9 (O3), U30.12 (B6)
- net ##105: now reaches U1.16 (O6)
- net ##105: now also J1.12 (Pin_12), U15.12 (D2), U25.3 (A1), U26.3 (A1), U27.18 (D7), U27.19 (O7), U28.19 (O7), U29.19 (O7), U30.17 (B1)
- net ##103: now reaches U1.17 (D6)
- net ##103: now also U24.19 (Pin_19)
- net ##102: now reaches U1.18 (D7)
- net ##102: now also U24.18 (Pin_18)
- net ##104: now reaches U1.19 (O7)
- net ##104: now also U15.13 (D3), U25.2 (A0), U26.2 (A0), U27.2 (O0), U27.3 (D0), U28.2 (O0), U29.2 (O0), U30.18 (B0)
- net ##121: now reaches U2.11 (B7)
- net ##121: now also U24.24 (Pin_24)
- net ##120: now reaches U2.12 (B6)
- net ##120: now also U24.25 (Pin_25)
- net ##119: now reaches U2.13 (B5)
- net ##119: now also U24.26 (Pin_26)
- net ##118: now reaches U2.14 (B4)
- net ##118: now also U24.27 (Pin_27)
- net ##117: now reaches U2.15 (B3)
- net ##117: now also U24.32 (Pin_32)
- net ##116: now reaches U2.16 (B2)
- net ##116: now also U24.33 (Pin_33)
- net ##115: now reaches U2.17 (B1)
- net ##115: now also U24.34 (Pin_34)
- net ##114: now reaches U2.18 (B0)
- net ##114: now also U24.35 (Pin_35)
- net GND: now reaches U2.19 (CE)
- net GND: now also J1.1 (Pin_1), J1.10 (Pin_10), J1.27 (Pin_27), J1.33 (Pin_33), J1.35 (Pin_35), J1.37 (Pin_37), J1.39 (Pin_39), J1.41 (Pin_41), J1.43 (Pin_43), J1.45 (Pin_45), J1.47 (Pin_47), J1.50 (Pin_50), U11.4 (E1), U11.5 (E2), U12.5 (E2), U18.2 (K), U21.10, U22.1 (Ea), U22.15 (Eb), U23.1 (Ea), U23.15 (Eb), U24.10 (Pin_10), U24.11 (Pin_11), U24.14 (Pin_14), U24.17 (Pin_17), U24.20 (Pin_20), U24.21 (Pin_21), U24.22 (Pin_22), U24.23 (Pin_23), U24.31 (Pin_31), U25.19 (CE), U31.8 (Pin_8), U31.9 (Pin_9), U44.15 (E), U45.1 (Ea), U45.15 (Eb), U46.1 (Ea), U46.15 (Eb), U55.1 (Ea), U55.11 (I1b), U55.15 (Eb), U55.6 (I0a), U58.15 (E), U61.15 (E), U62.A1 (NC), U62.D9 (GND), U62.E2 (GND), U62.G1 (VMA), U62.G2 (VPA), U62.K1 (NC), U62.K10 (NC), U63.A1 (NC), U63.D9 (GND), U63.E2 (GND), U63.K1 (NC), U63.K10 (NC), U64.8 (Pin_8), U64.9 (Pin_9), U65.8 (Pin_8), U65.9 (Pin_9)
- net ##122: now reaches U2.4 (A2)
- net ##122: now also J1.21 (Pin_21), U3.4 (A2), U4.16 (O6), U4.17 (D6), U5.16 (O6), U6.16 (O6), U7.6 (I2a), U8.14 (O2a)
- net ##123: now reaches U2.5 (A3)
- net ##123: now also J1.22 (Pin_22), U3.5 (A3), U30.11 (B7), U4.4 (D1), U4.5 (O1), U5.5 (O1), U6.5 (O1)
- net ##124: now reaches U2.6 (A4)
- net ##124: now also J1.23 (Pin_23), U3.6 (A4), U4.6 (O2), U4.7 (D2), U5.6 (O2), U6.6 (O2)
- net ##125: now reaches U2.7 (A5)
- net ##125: now also J1.24 (Pin_24), U3.7 (A5), U4.14 (D5), U4.15 (O5), U5.15 (O5), U6.15 (O5)
- net ##126: now reaches U2.8 (A6)
- net ##126: now also J1.25 (Pin_25), U3.8 (A6), U4.8 (D3), U4.9 (O3), U5.9 (O3), U6.9 (O3)
- net ##131: now reaches U3.1 (A->B)
- net ##131: now also J1.32 (Pin_32), U13.4 (E1), U26.1 (A->B), U30.1 (A->B), U40.9, U51.5, U72.12, U73.10
- net ##139: now reaches U3.11 (B7)
- net ##139: now also U62.B10 (D15), U63.B10 (D15)
- net ##138: now reaches U3.12 (B6)
- net ##138: now also U62.B9 (D14), U63.B9 (D14)
- net ##137: now reaches U3.13 (B5)
- net ##137: now also U62.C8 (D13), U63.C8 (D13)
- net ##136: now reaches U3.14 (B4)
- net ##136: now also U62.A10 (D12), U63.A10 (D12)
- net ##135: now reaches U3.15 (B3)
- net ##135: now also U62.B8 (D11), U63.B8 (D11)
- net ##134: now reaches U3.16 (B2)
- net ##134: now also U62.A9 (D10), U63.A9 (D10)
- net ##133: now reaches U3.17 (B1)
- net ##133: now also U62.B7 (D9), U63.B7 (D9)
- net ##132: now reaches U3.18 (B0)
- net ##132: now also U62.A8 (D8), U63.A8 (D8)
- net ##148: now reaches U4.1 (OE)
- net ##148: now also U27.1 (OE), U38.3
- net ##149: now reaches U4.11 (LE)
- net ##149: now also U27.11 (LE), U51.8
- net ##150: now reaches U5.1 (OE)
- net ##150: now also U14.10 (O5), U28.1 (OE)
- net ##151: now reaches U5.11 (LE)
- net ##151: now also U28.11 (LE), U29.11 (LE), U51.3, U70.2 (D)
- net A10: now reaches U5.17 (D6)
- net A10: now also U23.12 (I2b), U62.J8 (A10), U63.J8 (A10), U9.3
- net A9: now reaches U5.18 (D7)
- net A9: now also U23.4 (I2a), U62.K9 (A9), U63.K9 (A9), U9.4
- net A11: now reaches U5.4 (D1)
- net A11: now also U22.4 (I2a), U62.J9 (A11), U63.J9 (A11), U9.2
- net ##153: now reaches U6.1 (OE)
- net ##153: now also U14.12 (O3)
- net ##164: now reaches U6.11 (Cp)
- net ##164: now also U33.13, U68.9, U70.9 (Q)
- net ##163: now reaches U6.13 (D4)
- net ##163: now also U41.8
- net ##162: now reaches U6.14 (D5)
- net ##162: now also U10.8, U53.1
- net ##161: now reaches U6.17 (D6)
- net ##161: now also U33.6, U53.11, U53.12, U53.4
- net ##160: now reaches U6.18 (D7)
- net ##160: now also U52.11, U53.2
- net ##154: now reaches U6.3 (D0)
- net ##154: now also U14.4 (E1), U40.4, U51.9, U72.1, U72.4, U73.11, U73.8
- net ##155: now reaches U6.4 (D1)
- net ##155: now also U52.3, U53.3
- net ##156: now reaches U6.7 (D2)
- net ##156: now also U52.8, U53.6
- net ##157: now reaches U6.8 (D3)
- net ##157: now also U53.5, U68.11
- net ##166: now reaches U7.1 (OEa)
- net ##166: now also U31.10 (Pin_10), U41.2, U65.10 (Pin_10), U72.11
- net ##169: now reaches U7.11 (I0b)
- net ##169: now also U52.1, U7.8 (I3a), U71.6, U8.8 (I3a)
- net ##170: now reaches U7.12 (O3a)
- net ##170: now also U41.5, U64.14 (Pin_14), U7.9 (O0b)
- net ##175: now reaches U7.13 (I1b)
- net ##175: now also U17.15 (Q3)
- net ##168: now reaches U7.14 (O2a)
- net ##168: now also U17.13 (D3), U52.12, U64.11 (Pin_11), U66.4 (I), U7.7 (O1b), U8.6 (I2a)
- net ##176: now reaches U7.17 (I3b)
- net ##176: now also U72.6
- net ##167: now reaches U7.18 (O0a)
- net ##167: now also U17.12 (D2), U64.13 (Pin_13), U7.3 (O3b), U71.2, U8.2 (I0a)
- net ##177: now reaches U7.19 (OEb)
- net ##177: now also U33.12, U41.1
- net ##180: now reaches U8.1 (OEa)
- net ##180: now also U72.3
- net ISA_CLK: now reaches U8.11 (I0b)
- net ISA_CLK: now also J?.20 (CLK)
- net ##182: now reaches U8.15 (I2b)
- net ##182: now also J?.2 (RESET), U11.6 (E3), U16.10 (~S), U16.4 (~S), U35.10 (~S), U35.4 (~S), U47.1 (Pin_1), U54.1 (~R), U8.19 (OEb)
- net ISA_OSC: now reaches U8.17 (I3b)
- net ISA_OSC: now also J?.30 (OSC)
- net ##181: now reaches U8.5 (O2b)
- net ##181: now also U43.8
- net ##101: now reaches U8.7 (O1b)
- net ##101: now also U15.1 (~Mr), U16.14 (~R), U16.15 (~R), U20.14 (~R), U20.15 (~R), U24.12 (Pin_12), U35.1 (~R), U35.13 (~R), U36.1, U36.4, U54.4 (~S), U62.F2 (RESET), U63.F2 (RESET)
- net ##191: now reaches U9.12
- net ##191: now also U32.12
- net ##192: now reaches U9.8
- net ##192: now also U12.4 (E1), U13.5 (E2), U14.5 (E2), U48.1
- net ##200: now reaches U10.1
- net ##200: now also U13.6 (E3), U14.6 (E3), U16.1 (C), U16.13 (C), U17.1 (~Mr), U34.4, U39.13 (~R), U48.11, U51.1, U51.10, U51.4, U69.9 (Q)
- net ##165: now reaches U10.2
- net ##165: now also U29.13 (D4), U49.11, U62.C9 (A23), U63.C9 (A23), U67.10
- net ##201: now reaches U10.4
- net ##201: now also U15.7 (Q1), U49.10
- net ##202: now reaches U10.5
- net ##202: now also U49.9, U50.6
- net ##178: now reaches U10.6
- net ##178: now also U30.19 (CE), U72.13, U72.2
- net ##214: now reaches U10.10
- net ##214: now also U37.13
- net ##152: now reaches U10.12
- net ##152: now also U28.3 (D0), U52.10, U62.J4 (NC)
- net ##213: now reaches U10.13
- net ##213: now also U16.6 (~Q), U68.1
- net ##215: now reaches U10.9
- net ##215: now also U35.5 (Q), U38.9
- net ##225: now reaches U11.1 (A0)
- net ##225: now also U62.K3 (FC0), U63.K3 (FC0)
- net ##208: now reaches U11.10 (O5)
- net ##208: now also U48.3, U50.3
- net ##226: now reaches U11.2 (A1)
- net ##226: now also U62.J3 (FC1), U63.J3 (FC1)
- net ##212: now reaches U11.3 (A2)
- net ##212: now also U62.K2 (FC2), U63.J4 (NC), U67.5
- net ##233: now reaches U11.9 (O6)
- net ##233: now also U50.1
- net ##188: now reaches U12.6 (E3)
- net ##188: now also U18.4 (~S), U20.10 (~S), U20.4 (~S), U47.6 (Pin_6), U62.D1 (BR), U63.D1 (BR), U63.G2 (VPA), U63.H2 (IPL2), U63.H3 (IPL1), U63.J2 (IPL0)
- net ~ISA_IOW: now reaches J?.13 (~IOW)
- net ~ISA_IOW: now also U43.5
- net ~ISA_IOR: now reaches J?.14 (~IOR)
- net ~ISA_IOR: now also U42.1
- net ##276: now reaches J?.21 (IRQ7)
- net ##276: now also U21.6
- net ##247: now reaches U13.13 (O2)
- net ##247: now also U73.13
- net ##231: now reaches U13.7 (O7)
- net ##231: now also U54.2 (D), U68.4
- net ##248: now reaches U13.9 (O6)
- net ##248: now also U15.9 (Cp), U37.2, U37.5
- net ##158: now reaches U14.11 (O4)
- net ##158: now also U29.1 (OE)
- net ##256: now reaches U14.13 (O2)
- net ##256: now also U73.5
- net ##251: now reaches U14.7 (O7)
- net ##251: now also U38.1
- net ##234: now reaches U15.10 (Q2)
- net ##234: now also U34.10
- net ##209: now reaches U15.15 (Q3)
- net ##209: now also U48.5
- net ##205: now reaches U15.2 (Q0)
- net ##205: now also U33.3, U37.8
- net ##127: now reaches U15.4 (D0)
- net ##127: now also J1.13 (Pin_13), U25.4 (A2), U26.4 (A2), U27.16 (O6), U27.17 (D6), U28.16 (O6), U29.16 (O6), U30.16 (B2)
- net ##128: now reaches U15.5 (D1)
- net ##128: now also J1.14 (Pin_14), U25.5 (A3), U26.5 (A3), U27.4 (D1), U27.5 (O1), U28.5 (O1), U29.5 (O1), U30.15 (B3)
- net ##266: now reaches U16.2 (K)
- net ##266: now also U16.12 (K), U54.6 (~Q)
- net ##253: now reaches U16.3 (J)
- net ##253: now also U37.4
- net ##216: now reaches U16.5 (Q)
- net ##216: now also U33.10, U34.2, U40.2, U52.5
- net ##252: now reaches U16.11 (J)
- net ##252: now also U37.1
- net ##221: now reaches U16.7 (~Q)
- net ##221: now also U41.9, U48.10
- net ##262: now reaches U17.10 (Q2)
- net ##262: now also U72.5
- net ##222: now reaches U17.2 (Q0)
- net ##222: now also U39.2 (D), U48.9
- net ##265: now reaches U17.4 (D0)
- net ##265: now also U38.8
- net ##264: now reaches U17.5 (D1)
- net ##264: now also U38.11
- net ##270: now reaches U17.6 (~Q1)
- net ##270: now also U63.J1 (BERR)
- net ##246: now reaches U17.9 (Cp)
- net ##246: now also U39.11 (C), U52.4, U70.12 (D), U70.5 (Q)
- net ##250: now reaches U18.15 (~R)
- net ##250: now also U56.2, U70.13 (~R)
- net ##271: now reaches U18.5 (Q)
- net ##271: now also U40.13
- net ##272: now reaches U19.1 (~Mr)
- net ##272: now also U43.10
- net ##249: now reaches U19.7 (Q1)
- net ##249: now also U36.10, U36.13
- net ##277: now reaches U22.12 (I2b)
- net ##277: now also U44.12 (Zd)
- net ##279: now reaches U22.14 (S0)
- net ##279: now also J1.38 (Pin_38), U23.14 (S0), U45.14 (S0), U46.14 (S0)
- net ##278: now reaches U22.2 (S1)
- net ##278: now also J1.36 (Pin_36), U23.2 (S1), U45.2 (S1), U46.2 (S1), U61.1 (S)
- net ##95: now reaches U24.1 (Pin_1)
- net ##95: now also U25.16 (B2)
- net ##96: now reaches U24.2 (Pin_2)
- net ##96: now also U25.17 (B1)
- net ##97: now reaches U24.3 (Pin_3)
- net ##97: now also U25.18 (B0)
- net +5V: now reaches U24.30 (Pin_30)
- net +5V: now also U31.18 (Pin_18), U47.14 (Pin_14), U64.18 (Pin_18), U65.18 (Pin_18)
- net ##113: now reaches U24.36 (Pin_36)
- net ##113: now also U25.11 (B7)
- net ##112: now reaches U24.37 (Pin_37)
- net ##112: now also U25.12 (B6)
- net ##111: now reaches U24.38 (Pin_38)
- net ##111: now also U25.13 (B5)
- net ##110: now reaches U24.39 (Pin_39)
- net ##110: now also U25.14 (B4)
- net ##109: now reaches U24.40 (Pin_40)
- net ##109: now also U25.15 (B3)
- net ##100: now reaches U24.9 (Pin_9)
- net ##100: now also U67.11
- net ##129: now reaches U25.6 (A4)
- net ##129: now also J1.15 (Pin_15), U26.6 (A4), U27.6 (O2), U27.7 (D2), U28.6 (O2), U29.6 (O2), U30.14 (B4), U37.6
- net ##130: now reaches U25.7 (A5)
- net ##130: now also J1.16 (Pin_16), U26.7 (A5), U27.14 (D5), U27.15 (O5), U28.15 (O5), U29.15 (O5), U30.13 (B5), U37.3
- net ##147: now reaches U26.11 (B7)
- net ##147: now also U62.A7 (D7), U63.A7 (D7)
- net ##146: now reaches U26.12 (B6)
- net ##146: now also U62.B6 (D6), U63.B6 (D6)
- net ##145: now reaches U26.13 (B5)
- net ##145: now also U62.A6 (D5), U63.A6 (D5)
- net ##144: now reaches U26.14 (B4)
- net ##144: now also U62.A5 (D4), U63.A5 (D4)
- net ##143: now reaches U26.15 (B3)
- net ##143: now also U62.B5 (D3), U63.B5 (D3)
- net ##142: now reaches U26.16 (B2)
- net ##142: now also U62.A4 (D2), U63.A4 (D2)
- net ##141: now reaches U26.17 (B1)
- net ##141: now also U62.A3 (D1), U63.A3 (D1)
- net ##140: now reaches U26.18 (B0)
- net ##140: now also U62.B4 (D0), U63.B4 (D0)
- net ##159: now reaches U29.8 (D3)
- net ##159: now also U62.C10 (A22), U63.C10 (A22), U67.9
- net ##171: now reaches U30.6 (A4)
- net ##171: now also U58.13 (I1d), U65.14 (Pin_14), U66.1 (G)
- net ##172: now reaches U30.7 (A5)
- net ##172: now also U58.10 (I1c), U65.13 (Pin_13), U66.2 (H)
- net ##173: now reaches U30.8 (A6)
- net ##173: now also U58.6 (I1b), U65.12 (Pin_12), U66.13 (F)
- net ##174: now reaches U30.9 (A7)
- net ##174: now also U65.11 (Pin_11), U66.12 (E), U72.10
- net ##179: now reaches U64.10 (Pin_10)
- net ##179: now also U41.3, U41.4
- net ##194: now reaches U32.13
- net ##194: now also U33.11, U33.4, U34.1, U49.2, U50.5, U51.2, U67.6
- net ##183: now reaches U32.3
- net ##183: now also U40.11, U54.3 (C), U69.8 (~Q)
- net ##184: now reaches U32.4
- net ##184: now also U49.6
- net ##193: now reaches U32.6
- net ##193: now also J1.49 (Pin_49)
- net ##195: now reaches U32.10
- net ##195: now also U40.12
- net ##196: now reaches U32.8
- net ##196: now also U69.12 (D)
- net ##187: now reaches U32.9
- net ##187: now also U47.5 (Pin_5), U56.1, U56.3, U56.5, U62.A2 (AS), U63.A2 (AS)
- net ##203: now reaches U33.1
- net ##203: now also U39.8 (~Q), U49.5, U68.10
- net ##204: now reaches U33.2
- net ##204: now also U37.10, U44.1 (S), U52.13, U52.2, U58.1 (S), U68.13
- net ##206: now reaches U33.5
- net ##206: now also U72.8
- net ##218: now reaches U33.8
- net ##218: now also U38.2
- net ##217: now reaches U33.9
- net ##217: now also U51.6
- net ##227: now reaches U34.3
- net ##227: now also U49.3
- net ##220: now reaches U34.5
- net ##220: now also U48.12, U50.11
- net ##228: now reaches U34.6
- net ##228: now also U38.5
- net ##236: now reaches U34.8
- net ##236: now also U49.13
- net ##235: now reaches U34.9
- net ##235: now also U50.4
- net ##238: now reaches U35.2 (D)
- net ##238: now also U35.9 (Q), U36.5
- net ##239: now reaches U35.3 (C)
- net ##239: now also U36.12, U36.9, U73.4
- net ##240: now reaches U35.6 (~Q)
- net ##240: now also U38.13
- net ##232: now reaches U35.11 (C)
- net ##232: now also U68.6, U73.3
- net ##243: now reaches U35.12 (D)
- net ##243: now also U35.8 (~Q), U36.2
- net ##189: now reaches U36.3
- net ##189: now also U36.11, U47.7 (Pin_7), U63.C1 (BGACK), U63.F1 (HALT)
- net ##185: now reaches U36.6
- net ##185: now also U36.8, U47.3 (Pin_3), U62.C1 (BGACK), U62.F1 (HALT)
- net ##258: now reaches U37.11
- net ##258: now also U61.13 (I1d), U62.B2 (LDS), U63.B2 (LDS)
- net ##257: now reaches U37.12
- net ##257: now also U61.10 (I1c), U62.B3 (UDS), U63.B3 (UDS)
- net ##260: now reaches U38.4
- net ##260: now also J1.34 (Pin_34)
- net ##261: now reaches U38.6
- net ##261: now also U62.B1 (DTACK), U63.B1 (DTACK)
- net ##263: now reaches U38.10
- net ##263: now also U38.12, U39.12 (D), U41.10, U53.8
- net ##197: now reaches U39.1 (~R)
- net ##197: now also U39.10 (~S), U39.4 (~S), U47.13 (Pin_13)
- net ##267: now reaches U39.6 (~Q)
- net ##267: now also U62.J1 (BERR)
- net ##268: now reaches U39.9 (Q)
- net ##268: now also J1.44 (Pin_44)
- net ##237: now reaches U40.5
- net ##237: now also U68.8
- net ##230: now reaches U40.10
- net ##230: now also U68.3
- net ##259: now reaches U41.6
- net ##259: now also U71.13
- net ##273: now reaches U43.9
- net ##273: now also J1.42 (Pin_42)
- net ##186: now reaches U47.4 (Pin_4)
- net ##186: now also U62.H2 (IPL2)
- net ##199: now reaches U47.8 (Pin_8)
- net ##199: now also U70.10 (~S), U70.4 (~S)
- net ##198: now reaches U47.9 (Pin_9)
- net ##198: now also U69.1 (~R), U69.10 (~S), U69.4 (~S)
- net ##219: now reaches U48.13
- net ##219: now also U49.8
- net ##207: now reaches U48.2
- net ##207: now also U52.6
- net ##210: now reaches U48.6
- net ##210: now also U49.1
- net ##223: now reaches U48.8
- net ##223: now also U68.5
- net ##229: now reaches U49.4
- net ##229: now also U50.10
- net ##241: now reaches U50.2
- net ##241: now also U52.9
- net ##242: now reaches U54.11 (C)
- net ##242: now also U62.E1 (CLK), U63.E1 (CLK), U69.11 (C), U69.5 (Q), U70.3 (C)
- net ##245: now reaches U56.4
- net ##245: now also U70.1 (~R)
- net ##244: now reaches U56.6
- net ##244: now also U69.13 (~R)
- net ##211: now reaches U58.11 (I0c)
- net ##211: now also U67.3
- net ##274: now reaches U58.7 (Zb)
- net ##274: now also U61.6 (I1b)
- net ##275: now reaches U58.9 (Zc)
- net ##275: now also U61.3 (I1a)
- net ##280: now reaches U61.12 (Zd)
- net ##280: now also J1.31 (Pin_31)
- net ##281: now reaches U61.9 (Zc)
- net ##281: now also J1.30 (Pin_30)
- net ##269: now reaches U62.C3 (R/W)
- net ##269: now also U63.C3 (R/W), U73.9
- net ##190: now reaches U66.5 (Even)
- net ##190: now also U71.5
- net ##224: now reaches U67.8
- net ##224: now also U68.12, U72.9
- net ##254: now reaches U71.3
- net ##254: now also U71.12
- net ##255: now reaches U71.4
- net ##255: now also U71.11
- net #104: now reaches J1.11 (Pin_11)
- net ##33 renamed A12
- net ##34 renamed A13
- net ##35 renamed A14
- net ##36 renamed A15
- net ##37 renamed A16
- net ##38 renamed A17
- net ##39 renamed A18
- net ##40 renamed A19
- net ##41 renamed A20
- net ##42 renamed A21
- net ##67 renamed A7
- net ##68 renamed A8
- net ##69 renamed A5
- net ##70 renamed A6
- net ##71 renamed A1
- net ##72 renamed A2
- net ##73 renamed A3
- net ##74 renamed A4
- no-connect marks 0 -> 83
Other:
- moved on the sheet: J1, U18A, U18B, U19, U20A, U20B, U21A, U21B, U21C, U21D, U22, U23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
